File: SolidKey-1-PCB/SolidKey-1-PCB.kicad_pcb (KiCad board)
At the start: 2 copper layers, 276.8 x 105 mm, 220 parts, among them J101 USB_C_Receptacle_USB2.0_16P, J201 Conn_01x04, J202 Conn_01x02, J203 Conn_01x04, K301 TouchPoint, K302 TouchPoint, K303 TouchPoint, K304 TouchPoint, K305 TouchPoint, K306 TouchPoint, K307 TouchPoint, K308 TouchPoint, K309 TouchPoint, K310 TouchPoint, K311 TouchPoint, K312 TouchPoint, K313 TouchPoint, K314 TouchPoint, K315 TouchPoint, K316 TouchPoint, K401 TouchPoint, K402 TouchPoint, K403 TouchPoint, K404 TouchPoint, K405 TouchPoint, K406 TouchPoint, K407 TouchPoint, K408 TouchPoint, K409 TouchPoint, K410 TouchPoint, K411 TouchPoint, K412 TouchPoint, K413 TouchPoint, K414 TouchPoint, K415 TouchPoint, K416 TouchPoint, K501 TouchPoint, K502 TouchPoint, K503 TouchPoint, K504 TouchPoint, K505 TouchPoint, K506 TouchPoint, K507 TouchPoint, K508 TouchPoint, K509 TouchPoint, K510 TouchPoint, K511 TouchPoint, K512 TouchPoint, K513 TouchPoint, K514 TouchPoint, K515 TouchPoint, K516 TouchPoint, K601 TouchPoint, K602 TouchPoint, K603 TouchPoint, K604 TouchPoint, K605 TouchPoint, K606 TouchPoint, K607 TouchPoint, K608 TouchPoint, K609 TouchPoint, K610 TouchPoint, K611 TouchPoint, K612 TouchPoint, K613 TouchPoint, K614 TouchPoint, K615 TouchPoint, K616 TouchPoint, SW201 RUN/RESET, SW202 BOOT_SEL, U101 NCP1117-3.3_SOT223, U201 RP2040, U202 W25Q128JVS, U301 CY8CMBR3116, U401 CY8CMBR3116, U501 CY8CMBR3116, U601 CY8CMBR3116, Y201 ABM8-272-T3

Commit message: Add Framwork connectors and start routing
Parts:
- removed the K515 at (162.0, 422.5)
- removed the K515 at (262.0, 522.5)
- removed the K515 at (187.0, 472.5)
- removed the K515 at (237.0, 497.5)
- removed the K515 at (162.0, 472.5)
- removed the K515 at (212.0, 497.5)
- removed the K515 at (237.0, 522.5)
- removed the K515 at (237.0, 422.5)
- removed the K515 at (162.0, 447.5)
- removed the K515 at (187.0, 497.5)
- removed the K515 at (162.0, 522.5)
- removed the K515 at (262.0, 472.5)
- removed the K515 at (237.0, 447.5)
- removed the K515 at (187.0, 522.5)
- removed the K515 at (187.0, 422.5)
- removed the K515 at (212.0, 522.5)
- removed the K515 at (162.0, 497.5)
- removed the K515 at (212.0, 447.5)
- removed the K515 at (187.0, 447.5)
- removed the K515 at (212.0, 422.5)
- removed the K515 at (212.0, 472.5)
- removed the K515 at (262.0, 422.5)
- removed the K515 at (262.0, 447.5)
- removed the K515 at (237.0, 472.5)
- removed the K515 at (262.0, 497.5)
- removed R317, R417, R517, R617: 560, Resistor_SMD:R_0402_1005Metric
- added J701: Conn_01x10_MountingPin, SolidKey1_Footprints:046809610110846, B.Cu at (264.7, 26.2)
- added J702: Conn_01x10_MountingPin, SolidKey1_Footprints:046809610110846, B.Cu at (254.2, 42.5)
- added JP705: Jumper_2_Open, SolidKey1_Footprints:SolderJumper-2_P1.3mm_Open_XSilk_RoundedPad1.0x1.5mm, B.Cu at (271.9, 35.8)
- added JP706: Jumper_2_Open, SolidKey1_Footprints:SolderJumper-2_P1.3mm_Open_XSilk_RoundedPad1.0x1.5mm, B.Cu at (271.9, 39.8)
- added JP707: Jumper_2_Open, SolidKey1_Footprints:SolderJumper-2_P1.3mm_Open_XSilk_RoundedPad1.0x1.5mm, B.Cu at (271.9, 43.8)
- added K515: TouchPoint, SolidKey1_Footprints:KeySwitch1_General, F.Cu at (388.4, 210.8)
- added R105: 0, Resistor_SMD:R_0603_1608Metric, B.Cu at (287.8, 41.8)
- added R106: 0, Resistor_SMD:R_0603_1608Metric, B.Cu at (287.8, 40.0)
- added R701: 0, Resistor_SMD:R_0603_1608Metric, B.Cu at (276.2, 35.8)
- added R702: 0, Resistor_SMD:R_0603_1608Metric, B.Cu at (276.2, 39.5)
- added RU301: 3k3, Resistor_SMD:R_0402_1005Metric, B.Cu at (246.8, 56.1)
- added RU401: 3k3, Resistor_SMD:R_0402_1005Metric, B.Cu at (354.5, 233.8)
- added RU501: 3k3, Resistor_SMD:R_0402_1005Metric, F.Cu at (381.6, 220.1)
- added RU601: 3k3, Resistor_SMD:R_0402_1005Metric, B.Cu at (349.6, 229.8)
- D204: moved to F.Cu
- R306, R406, R506, R606: value 3k3 -> 560
- moved R309 338.3 mm to (414.2, -12.8)
- moved C102 315.1 mm to (288.0, 25.3), turned to 0 degrees
- moved C101 311.1 mm to (288.0, 27.6), turned to 0 degrees
- moved R103 301.4 mm to (288.2, 38.0)
- moved U101 300.6 mm to (282.1, 25.3)
- moved R104 298.3 mm to (288.5, 43.5)
- moved J101 298.2 mm to (294.9, 41.0), turned to -90 degrees
- moved R312 257.7 mm to (405.6, 57.7)
- moved K302 257.7 mm to (439.5, 27.3)
- moved K304 257.7 mm to (440.8, 73.7)
- moved K306 257.7 mm to (442.9, 117.0)
- moved K309 257.7 mm to (411.6, -0.50)
- moved R301 257.7 mm to (432.8, 9.60)
- moved R303 257.7 mm to (432.7, 60.3)
- moved R305 257.7 mm to (434.7, 105.9)
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Connections:
- J101 pad A6: /USB_DP -> Net-(J101-D+-PadA6)
- J101 pad A7: /USB_DM -> Net-(J101-D--PadA7)
- J101 pad B6: /USB_DP -> Net-(J101-D+-PadA6)
- J101 pad B7: /USB_DM -> Net-(J101-D--PadA7)
- R306 pad 1: /Cap_Sense_16_Channels_0/CAP_SENSE_HOST_INTERRUPT -> Net-(K306-Pad1)
- R306 pad 2: +3V3 -> Net-(U301-CS5)
- R307 pad 1: Net-(K306-Pad1) -> Net-(K307-Pad1)
- R307 pad 2: Net-(U301-CS5) -> Net-(U301-CS6)
- R308 pad 1: Net-(K307-Pad1) -> Net-(K308-Pad1)
- R308 pad 2: Net-(U301-CS6) -> Net-(U301-CS7)
- R309 pad 1: Net-(K308-Pad1) -> Net-(K309-Pad1)
- R309 pad 2: Net-(U301-CS7) -> Net-(U301-CS8)
- R310 pad 1: Net-(K309-Pad1) -> Net-(K310-Pad1)
- R310 pad 2: Net-(U301-CS8) -> Net-(U301-CS9)
- R311 pad 1: Net-(K310-Pad1) -> Net-(K311-Pad1)
- R311 pad 2: Net-(U301-CS9) -> Net-(U301-CS10)
- R312 pad 1: Net-(K311-Pad1) -> Net-(K312-Pad1)
- R312 pad 2: Net-(U301-CS10) -> Net-(U301-CS11)
- R313 pad 1: Net-(K312-Pad1) -> Net-(K313-Pad1)
- R313 pad 2: Net-(U301-CS11) -> Net-(U301-CS12)
- R314 pad 1: Net-(K313-Pad1) -> Net-(K314-Pad1)
- R314 pad 2: Net-(U301-CS12) -> Net-(U301-CS13)
- R315 pad 1: Net-(K314-Pad1) -> Net-(K315-Pad1)
- R315 pad 2: Net-(U301-CS13) -> Net-(U301-CS14)
- R316 pad 1: Net-(K315-Pad1) -> Net-(K316-Pad1)
- R316 pad 2: Net-(U301-CS14) -> Net-(U301-CS15)
- R406 pad 1: /Cap_Sense_16_Channels_1/CAP_SENSE_HOST_INTERRUPT -> Net-(K406-Pad1)
- R406 pad 2: +3V3 -> Net-(U401-CS5)
- R407 pad 1: Net-(K406-Pad1) -> Net-(K407-Pad1)
- R407 pad 2: Net-(U401-CS5) -> Net-(U401-CS6)
- R408 pad 1: Net-(K407-Pad1) -> Net-(K408-Pad1)
- R408 pad 2: Net-(U401-CS6) -> Net-(U401-CS7)
- R409 pad 1: Net-(K408-Pad1) -> Net-(K409-Pad1)
- R409 pad 2: Net-(U401-CS7) -> Net-(U401-CS8)
- R410 pad 1: Net-(K409-Pad1) -> Net-(K410-Pad1)
- R410 pad 2: Net-(U401-CS8) -> Net-(U401-CS9)
- R411 pad 1: Net-(K410-Pad1) -> Net-(K411-Pad1)
- R411 pad 2: Net-(U401-CS9) -> Net-(U401-CS10)
- R412 pad 1: Net-(K411-Pad1) -> Net-(K412-Pad1)
- R412 pad 2: Net-(U401-CS10) -> Net-(U401-CS11)
- R413 pad 1: Net-(K412-Pad1) -> Net-(K413-Pad1)
- R413 pad 2: Net-(U401-CS11) -> Net-(U401-CS12)
- R414 pad 1: Net-(K413-Pad1) -> Net-(K414-Pad1)
- R414 pad 2: Net-(U401-CS12) -> Net-(U401-CS13)
- R415 pad 1: Net-(K414-Pad1) -> Net-(K415-Pad1)
- R415 pad 2: Net-(U401-CS13) -> Net-(U401-CS14)
- R416 pad 1: Net-(K415-Pad1) -> Net-(K416-Pad1)
- R416 pad 2: Net-(U401-CS14) -> Net-(U401-CS15)
- R506 pad 1: /Cap_Sense_16_Channels_2/CAP_SENSE_HOST_INTERRUPT -> Net-(K506-Pad1)
- R506 pad 2: +3V3 -> Net-(U501-CS5)
- R507 pad 1: Net-(K506-Pad1) -> Net-(K507-Pad1)
- R507 pad 2: Net-(U501-CS5) -> Net-(U501-CS6)
- R508 pad 1: Net-(K507-Pad1) -> Net-(K508-Pad1)
- R508 pad 2: Net-(U501-CS6) -> Net-(U501-CS7)
- R509 pad 1: Net-(K508-Pad1) -> Net-(K509-Pad1)
- R509 pad 2: Net-(U501-CS7) -> Net-(U501-CS8)
- R510 pad 1: Net-(K509-Pad1) -> Net-(K510-Pad1)
- R510 pad 2: Net-(U501-CS8) -> Net-(U501-CS9)
- R511 pad 1: Net-(K510-Pad1) -> Net-(K511-Pad1)
- R511 pad 2: Net-(U501-CS9) -> Net-(U501-CS10)
- R512 pad 1: Net-(K511-Pad1) -> Net-(K512-Pad1)
- R512 pad 2: Net-(U501-CS10) -> Net-(U501-CS11)
- R513 pad 1: Net-(K512-Pad1) -> Net-(K513-Pad1)
- R513 pad 2: Net-(U501-CS11) -> Net-(U501-CS12)
- R514 pad 1: Net-(K513-Pad1) -> Net-(K514-Pad1)
- R514 pad 2: Net-(U501-CS12) -> Net-(U501-CS13)
- R515 pad 1: Net-(K514-Pad1) -> Net-(K515-Pad1)
- R515 pad 2: Net-(U501-CS13) -> Net-(U501-CS14)
- R516 pad 1: Net-(K515-Pad1) -> Net-(K516-Pad1)
- R516 pad 2: Net-(U501-CS14) -> Net-(U501-CS15)
- R606 pad 1: /Cap_Sense_16_Channels_3/CAP_SENSE_HOST_INTERRUPT -> Net-(K606-Pad1)
- R606 pad 2: +3V3 -> Net-(U601-CS5)
- R607 pad 1: Net-(K606-Pad1) -> Net-(K607-Pad1)
- R607 pad 2: Net-(U601-CS5) -> Net-(U601-CS6)
- R608 pad 1: Net-(K607-Pad1) -> Net-(K608-Pad1)
- R608 pad 2: Net-(U601-CS6) -> Net-(U601-CS7)
- R609 pad 1: Net-(K608-Pad1) -> Net-(K609-Pad1)
- R609 pad 2: Net-(U601-CS7) -> Net-(U601-CS8)
- R610 pad 1: Net-(K609-Pad1) -> Net-(K610-Pad1)
- R610 pad 2: Net-(U601-CS8) -> Net-(U601-CS9)
- R611 pad 1: Net-(K610-Pad1) -> Net-(K611-Pad1)
- R611 pad 2: Net-(U601-CS9) -> Net-(U601-CS10)
- R612 pad 1: Net-(K611-Pad1) -> Net-(K612-Pad1)
- R612 pad 2: Net-(U601-CS10) -> Net-(U601-CS11)
- R613 pad 1: Net-(K612-Pad1) -> Net-(K613-Pad1)
- R613 pad 2: Net-(U601-CS11) -> Net-(U601-CS12)
- R614 pad 1: Net-(K613-Pad1) -> Net-(K614-Pad1)
- R614 pad 2: Net-(U601-CS12) -> Net-(U601-CS13)
- R615 pad 1: Net-(K614-Pad1) -> Net-(K615-Pad1)
- R615 pad 2: Net-(U601-CS13) -> Net-(U601-CS14)
- R616 pad 1: Net-(K615-Pad1) -> Net-(K616-Pad1)
- R616 pad 2: Net-(U601-CS14) -> Net-(U601-CS15)
Routing:
- net /Microcontroller/GPIO18_LED: track 38.6 -> 131.5 mm
- net /USB_DP: track 0.00 -> 78.6 mm
- net +3V3: track 22.1 -> 91.3 mm
- net /USB_DM: track 0.00 -> 44.5 mm
- net /Framework_Connectors/FW_FINGERPRINT_P10: track 0.00 -> 33.0 mm
- net /Framework_Connectors/FW_FINGERPRINT_P09: track 0.00 -> 32.3 mm
- net VBUS: track 0.00 -> 32.1 mm
- net /Framework_Connectors/FW_FINGERPRINT_P08: track 0.00 -> 31.3 mm
- net /Framework_Connectors/FW_FINGERPRINT_P07: track 0.00 -> 30.6 mm
- net /Framework_Connectors/FW_FINGERPRINT_P06: track 0.00 -> 29.4 mm
- net /Framework_Connectors/FW_FINGERPRINT_P05: track 0.00 -> 28.6 mm
- net GND: track 0.00 -> 27.8 mm
- net /Framework_Connectors/FW_FINGERPRINT_P02: track 0.00 -> 26.7 mm
- net Net-(J702-Pin_1): track 0.00 -> 20.6 mm
- net Net-(J702-Pin_3): track 0.00 -> 19.7 mm
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- added copper zone on B.Cu, net VBUS
Other:
- board text added: "(20, 20) IS THIS CORNER"
- board text added: "FINGERPRINT/POWER BUTTON IS THIS CORNER"
- board text added: "To FP"
- board text added: "To MB"
- board text removed: ". <- (20, 20) IS HERE"

Commit message: Place each capacitive sensor chip block
Parts:
- removed J702: Conn_01x10_MountingPin, SolidKey1_Footprints:046809610110846
- K501: moved to F.Cu
- RU501: moved to B.Cu
- moved K416 455.2 mm to (-38.0, 30.0)
- moved K412 454.2 mm to (-54.6, 30.0)
- moved K408 453.2 mm to (-71.2, 30.0)
- moved K404 452.3 mm to (-87.7, 30.0)
- moved K415 448.8 mm to (-38.0, 13.4)
- moved K411 447.7 mm to (-54.6, 13.4)
- moved K407 446.8 mm to (-71.2, 13.4)
- moved K403 445.9 mm to (-87.7, 13.4)
- moved K414 442.4 mm to (-38.0, -3.10)
- moved K410 441.3 mm to (-54.6, -3.10)
- moved K406 440.3 mm to (-71.2, -3.10)
- moved K402 439.4 mm to (-87.7, -3.10)
- moved K413 436.0 mm to (-38.0, -19.6)
- moved K409 434.9 mm to (-54.6, -19.6)
- moved K405 433.9 mm to (-71.2, -19.6)
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Routing:
- net +3V3: track 91.3 -> 105.9 mm
- net Net-(U401-VCC): track 0.00 -> 2.12 mm
- net Net-(U601-VCC): track 0.00 -> 2.12 mm
- net Net-(U501-VCC): track 0.00 -> 2.12 mm
- net Net-(U401-CMOD): track 0.00 -> 1.87 mm
- net Net-(U601-CMOD): track 0.00 -> 1.87 mm
- net Net-(U501-CMOD): track 0.00 -> 1.87 mm
- net /Cap_Sense_16_Channels_3/CAP_SENSE_HOST_INTERRUPT: track 0.00 -> 1.34 mm
- net /Cap_Sense_16_Channels_2/CAP_SENSE_HOST_INTERRUPT: track 0.00 -> 1.34 mm
- net /Cap_Sense_16_Channels_1/CAP_SENSE_HOST_INTERRUPT: track 3.94 -> 5.27 mm
Other:
- board text removed: "To FP"
