File: SolidKey-1-PCB/SolidKey-1-PCB.kicad_pcb (KiCad board)
At the start: 2 copper layers, 276.8 x 105 mm, 204 parts, among them J101 USB_C_Receptacle_USB2.0_16P, J201 Conn_01x04, J202 Conn_01x02, J203 Conn_01x04, J701 Conn_01x10_MountingPin, K301 TouchPoint, K302 TouchPoint, K303 TouchPoint, K304 TouchPoint, K305 TouchPoint, K306 TouchPoint, K307 TouchPoint, K308 TouchPoint, K309 TouchPoint, K310 TouchPoint, K311 TouchPoint, K312 TouchPoint, K313 TouchPoint, K314 TouchPoint, K315 TouchPoint, K316 TouchPoint, K401 TouchPoint, K402 TouchPoint, K403 TouchPoint, K404 TouchPoint, K405 TouchPoint, K406 TouchPoint, K407 TouchPoint, K408 TouchPoint, K409 TouchPoint, K410 TouchPoint, K411 TouchPoint, K412 TouchPoint, K413 TouchPoint, K414 TouchPoint, K415 TouchPoint, K416 TouchPoint, K501 TouchPoint, K502 TouchPoint, K503 TouchPoint, K504 TouchPoint, K505 TouchPoint, K506 TouchPoint, K507 TouchPoint, K508 TouchPoint, K509 TouchPoint, K510 TouchPoint, K511 TouchPoint, K512 TouchPoint, K513 TouchPoint, K514 TouchPoint, K515 TouchPoint, K516 TouchPoint, K601 TouchPoint, K602 TouchPoint, K603 TouchPoint, K604 TouchPoint, K605 TouchPoint, K606 TouchPoint, K607 TouchPoint, K608 TouchPoint, K609 TouchPoint, K610 TouchPoint, K611 TouchPoint, K612 TouchPoint, K613 TouchPoint, K614 TouchPoint, K615 TouchPoint, K616 TouchPoint, SW201 RUN/RESET, SW202 BOOT_SEL, U101 NCP1117-3.3_SOT223, U201 RP2040, U202 W25Q128JVS, U301 CY8CMBR3116, U401 CY8CMBR3116, U501 CY8CMBR3116, U601 CY8CMBR3116, Y201 ABM8-272-T3

Commit message: Prepare to place the keys
Parts:
- added J702: Conn_01x10_MountingPin, SolidKey1_Footprints:046809610110846, B.Cu at (254.3, 42.5)
- moved K301 370.6 mm to (29.6, 37.4)
Other:
- board text added: "To FP"

Commit message: Finish key layout placement
Parts:
- moved K304 370.7 mm to (29.6, 88.9)
- moved K303 370.7 mm to (29.6, 71.7)
- moved K302 370.7 mm to (29.6, 54.5)
- moved K308 370.1 mm to (46.8, 88.9)
- moved K307 370.0 mm to (46.8, 71.7)
- moved K306 370.0 mm to (46.8, 54.5)
- moved K305 370.0 mm to (46.8, 37.3)
- moved K312 369.3 mm to (64.0, 84.6)
- moved K311 369.3 mm to (64.0, 67.4)
- moved K310 369.2 mm to (64.0, 50.2)
- moved K309 369.2 mm to (64.0, 33.0)
- moved K316 368.6 mm to (81.2, 82.4)
- moved K315 368.5 mm to (81.2, 65.2)
- moved K314 368.5 mm to (81.2, 48.0)
- moved K313 368.5 mm to (81.2, 30.8)
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
Commit message: Reposition CapSense chips
Parts:
- R301, R302, R303, R304, R305, R306, R307, R308, R309, R310, R311, R312, R313, R314, R315, R316, R401, R402, R403, R404, R405, R406, R407, R408, R409, R410, R411, R412, R413, R414, R415, R416, R501, R502, R503, R504, R505, R506, R507, R508, R509, R510, R511, R512, R513, R514, R515, R516, R601, R602, R603, R604, R605, R606, R607, R608, R609, R610, R611, R612, R613, R614, R615, R616: footprint Resistor_SMD:R_0402_1005Metric -> Resistor_SMD:R_0603_1608Metric
- moved R301 372.7 mm to (-10.8, 56.0)
- moved R302 372.7 mm to (-10.8, 58.0)
- moved R303 372.7 mm to (-10.8, 60.0)
- moved R304 372.7 mm to (-10.8, 62.0)
- moved R305 372.7 mm to (-7.91, 56.0)
- moved R306 372.7 mm to (-7.91, 58.0)
- moved R307 372.7 mm to (-7.91, 60.0)
- moved R308 372.7 mm to (-7.91, 62.0)
- moved R309 372.7 mm to (-5.00, 56.0)
- moved R310 372.7 mm to (-5.00, 58.0)
- moved R311 372.7 mm to (-5.00, 60.0)
- moved R312 372.7 mm to (-5.00, 62.0)
- moved R313 372.7 mm to (-2.09, 56.0)
- moved R314 372.7 mm to (-2.09, 58.0)
- moved R315 372.7 mm to (-2.09, 60.0)
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Routing:
- net +3V3: track 105.9 -> 102.3 mm
