File: SolidKey-1-PCB/Cap_Sense_16_Channels.kicad_sch (KiCad schematic)
At the start: 38 parts, among them K501 TouchPoint, K502 TouchPoint, K503 TouchPoint, K504 TouchPoint, K505 TouchPoint, K506 TouchPoint, K507 TouchPoint, K508 TouchPoint, K509 TouchPoint, K510 TouchPoint, K511 TouchPoint, K512 TouchPoint, K513 TouchPoint, K514 TouchPoint, K515 TouchPoint, K516 TouchPoint, U501 CY8CMBR3116

Commit message: Add Framwork connectors and start routing
Parts:
- renumbered R507 to R506, R508 to R507, R509 to R508, R510 to R509, R511 to R510, R512 to R511, R513 to R512, R514 to R513, R515 to R514, R516 to R515, R517 to R516, R506 to RU501
Changed lines of the file:
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@@
 		(on_board yes)
 		(dnp no)
-		(property "Reference" "R514"
+		(property "Reference" "R513"
 			(at 96.774 96.774 90)
 			(effects
@@
 			(project "SolidKey-1-PCB"
 				(path "/ab9c01e5-18ba-437e-8193-74ebfda4cffd/0985ec50-8c81-46bb-8805-f9fa10785c64"
-					(reference "R514")
+					(reference "R513")
 					(unit 1)
 				)
 				(path "/ab9c01e5-18ba-437e-8193-74ebfda4cffd/47acc2ae-bd18-4aee-bff6-1b0674fb2f64"
-					(reference "R314")
+					(reference "R313")
 					(unit 1)
 				)
 				(path "/ab9c01e5-18ba-437e-8193-74ebfda4cffd/a2b4e060-f2e7-4c89-a69e-4749e8ac3539"
-					(reference "R414")
+					(reference "R413")
 					(unit 1)
 				)
 				(path "/ab9c01e5-18ba-437e-8193-74ebfda4cffd/d81672ba-5fbd-4dc8-920d-12fa7a286f16"
-					(reference "R614")
+					(reference "R613")
 					(unit 1)
 				)
@@
 		(on_board yes)
 		(dnp no)
-		(property "Reference" "R517"
+		(property "Reference" "R516"
 			(at 96.774 104.394 90)
 			(effects
@@
 					(size 1.27 1.27)
 				)
-				(hide yes)
 			)
 		)
@@
 			(project "SolidKey-1-PCB"
 				(path "/ab9c01e5-18ba-437e-8193-74ebfda4cffd/0985ec50-8c81-46bb-8805-f9fa10785c64"
-					(reference "R517")
+					(reference "R516")
 					(unit 1)
 				)
 				(path "/ab9c01e5-18ba-437e-8193-74ebfda4cffd/47acc2ae-bd18-4aee-bff6-1b0674fb2f64"
-					(reference "R317")
+					(reference "R316")
 					(unit 1)
 				)
 				(path "/ab9c01e5-18ba-437e-8193-74ebfda4cffd/a2b4e060-f2e7-4c89-a69e-4749e8ac3539"
-					(reference "R417")
+					(reference "R416")
 					(unit 1)
 				)
 				(path "/ab9c01e5-18ba-437e-8193-74ebfda4cffd/d81672ba-5fbd-4dc8-920d-12fa7a286f16"
-					(reference "R617")
+					(reference "R616")
 					(unit 1)
 				)
@@
 		(on_board yes)
 		(dnp no)
-		(property "Reference" "R512"
+		(property "Reference" "R511"
 			(at 97.028 91.694 90)
 			(effects
@@
 			(project "SolidKey-1-PCB"
 				(path "/ab9c01e5-18ba-437e-8193-74ebfda4cffd/0985ec50-8c81-46bb-8805-f9fa10785c64"
-					(reference "R512")
+					(reference "R511")
 					(unit 1)
 				)
 				(path "/ab9c01e5-18ba-437e-8193-74ebfda4cffd/47acc2ae-bd18-4aee-bff6-1b0674fb2f64"
-					(reference "R312")
+					(reference "R311")
 					(unit 1)
 				)
 				(path "/ab9c01e5-18ba-437e-8193-74ebfda4cffd/a2b4e060-f2e7-4c89-a69e-4749e8ac3539"
-					(reference "R412")
+					(reference "R411")
 					(unit 1)
 				)
 				(path "/ab9c01e5-18ba-437e-8193-74ebfda4cffd/d81672ba-5fbd-4dc8-920d-12fa7a286f16"
-					(reference "R612")
+					(reference "R611")
 					(unit 1)
 				)
@@
 		(on_board yes)
 		(dnp no)
-		(property "Reference" "R509"
+		(property "Reference" "R508"
 			(at 97.536 83.82 90)
 			(effects
@@
 			(project "SolidKey-1-PCB"
 				(path "/ab9c01e5-18ba-437e-8193-74ebfda4cffd/0985ec50-8c81-46bb-8805-f9fa10785c64"
-					(reference "R509")
+					(reference "R508")
 					(unit 1)
 				)
 				(path "/ab9c01e5-18ba-437e-8193-74ebfda4cffd/47acc2ae-bd18-4aee-bff6-1b0674fb2f64"
-					(reference "R309")
+					(reference "R308")
 					(unit 1)
 				)
 				(path "/ab9c01e5-18ba-437e-8193-74ebfda4cffd/a2b4e060-f2e7-4c89-a69e-4749e8ac3539"
-					(reference "R409")
+					(reference "R408")
 					(unit 1)
 				)
 				(path "/ab9c01e5-18ba-437e-8193-74ebfda4cffd/d81672ba-5fbd-4dc8-920d-12fa7a286f16"
-					(reference "R609")
+					(reference "R608")
 					(unit 1)
 				)
@@
 		(on_board yes)
 		(dnp no)
-		(property "Reference" "R515"
+		(property "Reference" "R514"
 			(at 96.774 99.314 90)
 			(effects
@@
 			(project "SolidKey-1-PCB"
 				(path "/ab9c01e5-18ba-437e-8193-74ebfda4cffd/0985ec50-8c81-46bb-8805-f9fa10785c64"
-					(reference "R515")
+					(reference "R514")
 					(unit 1)
 				)
 				(path "/ab9c01e5-18ba-437e-8193-74ebfda4cffd/47acc2ae-bd18-4aee-bff6-1b0674fb2f64"
-					(reference "R315")
+					(reference "R314")
 					(unit 1)
 				)
 				(path "/ab9c01e5-18ba-437e-8193-74ebfda4cffd/a2b4e060-f2e7-4c89-a69e-4749e8ac3539"
-					(reference "R415")
+					(reference "R414")
 					(unit 1)
 				)
 				(path "/ab9c01e5-18ba-437e-8193-74ebfda4cffd/d81672ba-5fbd-4dc8-920d-12fa7a286f16"
-					(reference "R615")
+					(reference "R614")
 					(unit 1)
 				)
@@
 		(on_board yes)
 		(dnp no)
-		(property "Reference" "R511"
+		(property "Reference" "R510"
 			(at 97.028 89.154 90)
 			(effects
@@
 			(project "SolidKey-1-PCB"
 				(path "/ab9c01e5-18ba-437e-8193-74ebfda4cffd/0985ec50-8c81-46bb-8805-f9fa10785c64"
-					(reference "R511")
+					(reference "R510")
 					(unit 1)
 				)
 				(path "/ab9c01e5-18ba-437e-8193-74ebfda4cffd/47acc2ae-bd18-4aee-bff6-1b0674fb2f64"
-					(reference "R311")
+					(reference "R310")
 					(unit 1)
 				)
 				(path "/ab9c01e5-18ba-437e-8193-74ebfda4cffd/a2b4e060-f2e7-4c89-a69e-4749e8ac3539"
-					(reference "R411")
+					(reference "R410")
 					(unit 1)
 				)
 				(path "/ab9c01e5-18ba-437e-8193-74ebfda4cffd/d81672ba-5fbd-4dc8-920d-12fa7a286f16"
-					(reference "R611")
+					(reference "R610")
 					(unit 1)
 				)
@@
 		(on_board yes)
 		(dnp no)
-		(property "Reference" "R507"
+		(property "Reference" "R506"
 			(at 97.536 78.74 90)
 			(effects
@@
 			(project "SolidKey-1-PCB"
 				(path "/ab9c01e5-18ba-437e-8193-74ebfda4cffd/0985ec50-8c81-46bb-8805-f9fa10785c64"
-					(reference "R507")
+					(reference "R506")
 					(unit 1)
 				)
 				(path "/ab9c01e5-18ba-437e-8193-74ebfda4cffd/47acc2ae-bd18-4aee-bff6-1b0674fb2f64"
-					(reference "R307")
+					(reference "R306")
 					(unit 1)
 				)
 				(path "/ab9c01e5-18ba-437e-8193-74ebfda4cffd/a2b4e060-f2e7-4c89-a69e-4749e8ac3539"
-					(reference "R407")
+					(reference "R406")
 					(unit 1)
 				)
 				(path "/ab9c01e5-18ba-437e-8193-74ebfda4cffd/d81672ba-5fbd-4dc8-920d-12fa7a286f16"
-					(reference "R607")
+					(reference "R606")
 					(unit 1)
 				)
@@
 		(on_board yes)
 		(dnp no)
-		(property "Reference" "R506"
+		(property "Reference" "RU501"
 			(at 181.61 74.168 90)
 			(effects
@@
 			(project ""
 				(path "/ab9c01e5-18ba-437e-8193-74ebfda4cffd/0985ec50-8c81-46bb-8805-f9fa10785c64"
-					(reference "R506")
+					(reference "RU501")
 					(unit 1)
 				)
 				(path "/ab9c01e5-18ba-437e-8193-74ebfda4cffd/47acc2ae-bd18-4aee-bff6-1b0674fb2f64"
-					(reference "R306")
+					(reference "RU301")
 					(unit 1)
 				)
 				(path "/ab9c01e5-18ba-437e-8193-74ebfda4cffd/a2b4e060-f2e7-4c89-a69e-4749e8ac3539"
-					(reference "R406")
+					(reference "RU401")
 					(unit 1)
 				)
 				(path "/ab9c01e5-18ba-437e-8193-74ebfda4cffd/d81672ba-5fbd-4dc8-920d-12fa7a286f16"
-					(reference "R606")
+					(reference "RU601")
 					(unit 1)
 				)
@@
 		(on_board yes)
 		(dnp no)
-		(property "Reference" "R516"
+		(property "Reference" "R515"
 			(at 96.774 101.854 90)
 			(effects
@@
 			(project "SolidKey-1-PCB"
 				(path "/ab9c01e5-18ba-437e-8193-74ebfda4cffd/0985ec50-8c81-46bb-8805-f9fa10785c64"
-					(reference "R516")
+					(reference "R515")
 					(unit 1)
 				)
 				(path "/ab9c01e5-18ba-437e-8193-74ebfda4cffd/47acc2ae-bd18-4aee-bff6-1b0674fb2f64"
-					(reference "R316")
+					(reference "R315")
 					(unit 1)
 				)
 				(path "/ab9c01e5-18ba-437e-8193-74ebfda4cffd/a2b4e060-f2e7-4c89-a69e-4749e8ac3539"
-					(reference "R416")
+					(reference "R415")
 					(unit 1)
 				)
 				(path "/ab9c01e5-18ba-437e-8193-74ebfda4cffd/d81672ba-5fbd-4dc8-920d-12fa7a286f16"
-					(reference "R616")
+					(reference "R615")
 					(unit 1)
 				)
@@
 		(on_board yes)
 		(dnp no)
-		(property "Reference" "R508"
+		(property "Reference" "R507"
 			(at 97.536 81.28 90)
 			(effects
@@
 			(project "SolidKey-1-PCB"
 				(path "/ab9c01e5-18ba-437e-8193-74ebfda4cffd/0985ec50-8c81-46bb-8805-f9fa10785c64"
-					(reference "R508")
+					(reference "R507")
 					(unit 1)
 				)
 				(path "/ab9c01e5-18ba-437e-8193-74ebfda4cffd/47acc2ae-bd18-4aee-bff6-1b0674fb2f64"
-					(reference "R308")
+					(reference "R307")
 					(unit 1)
 				)
 				(path "/ab9c01e5-18ba-437e-8193-74ebfda4cffd/a2b4e060-f2e7-4c89-a69e-4749e8ac3539"
-					(reference "R408")
+					(reference "R407")
 					(unit 1)
 				)
 				(path "/ab9c01e5-18ba-437e-8193-74ebfda4cffd/d81672ba-5fbd-4dc8-920d-12fa7a286f16"
-					(reference "R608")
+					(reference "R607")
 					(unit 1)
 				)
@@
 		(on_board yes)
 		(dnp no)
-		(property "Reference" "R513"
+		(property "Reference" "R512"
 			(at 96.774 94.234 90)
 			(effects
@@
 			(project "SolidKey-1-PCB"
 				(path "/ab9c01e5-18ba-437e-8193-74ebfda4cffd/0985ec50-8c81-46bb-8805-f9fa10785c64"
-					(reference "R513")
+					(reference "R512")
 					(unit 1)
 				)
 				(path "/ab9c01e5-18ba-437e-8193-74ebfda4cffd/47acc2ae-bd18-4aee-bff6-1b0674fb2f64"
-					(reference "R313")
+					(reference "R312")
 					(unit 1)
 				)
 				(path "/ab9c01e5-18ba-437e-8193-74ebfda4cffd/a2b4e060-f2e7-4c89-a69e-4749e8ac3539"
-					(reference "R413")
+					(reference "R412")
 					(unit 1)
 				)
 				(path "/ab9c01e5-18ba-437e-8193-74ebfda4cffd/d81672ba-5fbd-4dc8-920d-12fa7a286f16"
-					(reference "R613")
+					(reference "R612")
 					(unit 1)
 				)
@@
 		(on_board yes)
 		(dnp no)
-		(property "Reference" "R510"
+		(property "Reference" "R509"
 			(at 97.536 86.36 90)
 			(effects
@@
 			(project "SolidKey-1-PCB"
 				(path "/ab9c01e5-18ba-437e-8193-74ebfda4cffd/0985ec50-8c81-46bb-8805-f9fa10785c64"
-					(reference "R510")
+					(reference "R509")
 					(unit 1)
 				)
 				(path "/ab9c01e5-18ba-437e-8193-74ebfda4cffd/47acc2ae-bd18-4aee-bff6-1b0674fb2f64"
-					(reference "R310")
+					(reference "R309")
 					(unit 1)
 				)
 				(path "/ab9c01e5-18ba-437e-8193-74ebfda4cffd/a2b4e060-f2e7-4c89-a69e-4749e8ac3539"
-					(reference "R410")
+					(reference "R409")
 					(unit 1)
 				)
 				(path "/ab9c01e5-18ba-437e-8193-74ebfda4cffd/d81672ba-5fbd-4dc8-920d-12fa7a286f16"
-					(reference "R610")
+					(reference "R609")
 					(unit 1)
 				)

Commit message: Reposition CapSense chips
Parts:
- R501, R502, R503, R504, R505, R506, R507, R508, R509, R510, R511, R512, R513, R514, R515, R516: footprint Resistor_SMD:R_0402_1005Metric -> Resistor_SMD:R_0603_1608Metric
Other:
- note added: "Place resistors close to chip"
Changed lines of the file:
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@@
 		)
 	)
+	(text "Place resistors close to chip"
+		(exclude_from_sim no)
+		(at 95.758 62.484 0)
+		(effects
+			(font
+				(size 1.27 1.27)
+			)
+		)
+	)
 	(text "VCC: Internal Regulator Output"
 		(exclude_from_sim no)
@@
 			)
 		)
-		(property "Footprint" "Resistor_SMD:R_0402_1005Metric"
+		(property "Footprint" "Resistor_SMD:R_0603_1608Metric"
 			(at 101.6 99.568 90)
 			(effects
@@
 			)
 		)
-		(property "Footprint" "Resistor_SMD:R_0402_1005Metric"
+		(property "Footprint" "Resistor_SMD:R_0603_1608Metric"
 			(at 101.6 69.088 90)
 			(effects
@@
 			)
 		)
-		(property "Footprint" "Resistor_SMD:R_0402_1005Metric"
+		(property "Footprint" "Resistor_SMD:R_0603_1608Metric"
 			(at 101.6 107.188 90)
 			(effects
@@
 			)
 		)
-		(property "Footprint" "Resistor_SMD:R_0402_1005Metric"
+		(property "Footprint" "Resistor_SMD:R_0603_1608Metric"
 			(at 101.6 94.488 90)
 			(effects
@@
 			)
 		)
-		(property "Footprint" "Resistor_SMD:R_0402_1005Metric"
+		(property "Footprint" "Resistor_SMD:R_0603_1608Metric"
 			(at 101.6 86.868 90)
 			(effects
@@
 			)
 		)
-		(property "Footprint" "Resistor_SMD:R_0402_1005Metric"
+		(property "Footprint" "Resistor_SMD:R_0603_1608Metric"
 			(at 101.6 71.628 90)
 			(effects
@@
 			)
 		)
-		(property "Footprint" "Resistor_SMD:R_0402_1005Metric"
+		(property "Footprint" "Resistor_SMD:R_0603_1608Metric"
 			(at 101.6 102.108 90)
 			(effects
@@
 			)
 		)
-		(property "Footprint" "Resistor_SMD:R_0402_1005Metric"
+		(property "Footprint" "Resistor_SMD:R_0603_1608Metric"
 			(at 101.6 74.168 90)
 			(effects
@@
 			)
 		)
-		(property "Footprint" "Resistor_SMD:R_0402_1005Metric"
+		(property "Footprint" "Resistor_SMD:R_0603_1608Metric"
 			(at 101.6 91.948 90)
 			(effects
@@
 			)
 		)
-		(property "Footprint" "Resistor_SMD:R_0402_1005Metric"
+		(property "Footprint" "Resistor_SMD:R_0603_1608Metric"
 			(at 101.6 81.788 90)
 			(effects
@@
 			)
 		)
-		(property "Footprint" "Resistor_SMD:R_0402_1005Metric"
+		(property "Footprint" "Resistor_SMD:R_0603_1608Metric"
 			(at 101.6 76.708 90)
 			(effects
@@
 			)
 		)
-		(property "Footprint" "Resistor_SMD:R_0402_1005Metric"
+		(property "Footprint" "Resistor_SMD:R_0603_1608Metric"
 			(at 101.6 104.648 90)
 			(effects
@@
 			)
 		)
-		(property "Footprint" "Resistor_SMD:R_0402_1005Metric"
+		(property "Footprint" "Resistor_SMD:R_0603_1608Metric"
 			(at 101.6 79.248 90)
 			(effects
@@
 			)
 		)
-		(property "Footprint" "Resistor_SMD:R_0402_1005Metric"
+		(property "Footprint" "Resistor_SMD:R_0603_1608Metric"
 			(at 101.6 84.328 90)
 			(effects
@@
 			)
 		)
-		(property "Footprint" "Resistor_SMD:R_0402_1005Metric"
+		(property "Footprint" "Resistor_SMD:R_0603_1608Metric"
 			(at 101.6 97.028 90)
 			(effects
@@
 			)
 		)
-		(property "Footprint" "Resistor_SMD:R_0402_1005Metric"
+		(property "Footprint" "Resistor_SMD:R_0603_1608Metric"
 			(at 101.6 89.408 90)
 			(effects
